File: hardware/Test_Boards/BlankHat/BlankHat.kicad_sch (KiCad schematic)
At the start: 9 parts, among them J1 Conn_01x08_Socket, J2 Conn_01x08_Socket, J3 Conn_01x08_Socket, Q1 PZT2222A, U1 74HC688, U2 74HC245, U3 74HC245

Commit message: started working on blank smd hat:
Parts:
- removed Q1: PZT2222A, Package_TO_SOT_SMD:SOT-223-3_TabPin2, symbol Transistor_BJT:PZT2222A
- removed R1, R2: 1k, Resistor_SMD:R_0201_0603Metric, symbol Device:R
- U1, U2, U3: footprint Package_SO:TSSOP-20_4.4x6.5mm_P0.65mm -> Package_DIP:DIP-20_W7.62mm
Connections:
- net D15 is gone; now on net D7: U3.18 (B0)
- net RESP is gone; now on net I5: J1.7 (Pin_7)
- net +5V: now also U2.2 (A0)
- net D0: now also U2.17 (B1); no longer U2.11 (B7)
- net D1: now also U2.16 (B2); no longer U2.12 (B6)
- net D10: now also U3.15 (B3); no longer U3.13 (B5)
- net D12: now also U3.13 (B5); no longer U3.15 (B3)
- net D13: now also U3.12 (B6); no longer U3.16 (B2)
- net D14: now also U3.11 (B7); no longer U3.17 (B1)
- net D2: now also U2.15 (B3); no longer U2.13 (B5)
- net D4: now also U2.13 (B5); no longer U2.15 (B3)
- net D5: now also U2.12 (B6); no longer U2.16 (B2)
- net D6: now also U2.11 (B7); no longer U2.17 (B1)
- net D7: no longer U2.18 (B0)
- net D8: now also U3.17 (B1); no longer U3.11 (B7)
- net D9: now also U3.16 (B2); no longer U3.12 (B6)
- net at J2.1 (Pin_1): now also U2.18 (B0); no longer U2.2 (A0)
