File: hardware/MainBoard/MainBoard.kicad_pcb (KiCad board)
At the start: 2 copper layers, 38.1 x 101.6 mm, 4 parts, among them J1 Conn_01x08_Socket, J2 Conn_01x08_Socket, J3 Conn_01x08_Socket, U1 ESP32-S3-WROOM-1

Commit message: added more stuff to main board
Parts:
- added BZ1: Buzzer, Buzzer_Beeper:Buzzer_Mallory_AST1109MLTRQ, F.Cu at (70.5, 83.0)
- added J4: Micro_SD_Card_Det2, Connector_Card:microSD_HC_Hirose_DM3AT-SF-PEJM5, F.Cu at (59.6, 96.4)
- added P1: USB_C_Plug_USB2.0, Connector_USB:USB_C_Receptacle_Amphenol_12401610E4-2A, F.Cu at (56.5, 83.1)
- J1, J2, J3: moved to B.Cu
- moved U1 48.5 mm to (70.0, 63.7), turned to 0 degrees
- moved J1 17.8 mm to (78.7, 150.6)
- turned J2 to 180 degrees
- turned J3 to 0 degrees
Other:
- board text added: "T.A.C.O.S Main Board"

Commit message: finished usb and voltage regulator
Connections:
- P1 pad A6: unconnected-(P1-D+-PadA6) -> USB+
- P1 pad A7: unconnected-(P1-D--PadA7) -> USB-
- U1 pad 13: unconnected-(U1-USB_D--Pad13) -> USB-
- U1 pad 14: unconnected-(U1-USB_D+-Pad14) -> USB+
Changed lines of the file:
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@@
 	(net 55 "unconnected-(U1-IO46-Pad16)")
 	(net 56 "unconnected-(U1-IO47-Pad24)")
-	(net 57 "unconnected-(U1-USB_D+-Pad14)")
-	(net 58 "unconnected-(U1-IO11-Pad19)")
-	(net 59 "unconnected-(U1-IO21-Pad23)")
-	(net 60 "unconnected-(U1-IO10-Pad18)")
-	(net 61 "unconnected-(U1-USB_D--Pad13)")
-	(net 62 "unconnected-(U1-IO45-Pad26)")
-	(net 63 "unconnected-(U1-IO39-Pad32)")
-	(net 64 "unconnected-(J4-DAT1-Pad8)")
-	(net 65 "unconnected-(J4-SHIELD-Pad11)")
-	(net 66 "unconnected-(J4-DAT3{slash}CD-Pad2)")
-	(net 67 "unconnected-(J4-CMD-Pad3)")
-	(net 68 "unconnected-(J4-DAT0-Pad7)")
-	(net 69 "unconnected-(J4-DAT2-Pad1)")
-	(net 70 "unconnected-(J4-DET_A-Pad10)")
-	(net 71 "unconnected-(J4-CLK-Pad5)")
-	(net 72 "unconnected-(J4-VDD-Pad4)")
-	(net 73 "unconnected-(J4-DET_B-Pad9)")
-	(net 74 "unconnected-(J4-VSS-Pad6)")
-	(net 75 "unconnected-(BZ1-+-Pad1)")
-	(net 76 "unconnected-(BZ1---Pad2)")
-	(net 77 "Net-(P1-VBUS-PadA4)")
-	(net 78 "Net-(P1-GND-PadA1)")
-	(net 79 "unconnected-(P1-CC-PadA5)")
-	(net 80 "unconnected-(P1-SHIELD-PadS1)")
-	(net 81 "unconnected-(P1-D+-PadA6)")
-	(net 82 "unconnected-(P1-VCONN-PadB5)")
-	(net 83 "unconnected-(P1-D--PadA7)")
+	(net 57 "unconnected-(U1-IO11-Pad19)")
+	(net 58 "unconnected-(U1-IO21-Pad23)")
+	(net 59 "unconnected-(U1-IO10-Pad18)")
+	(net 60 "unconnected-(U1-IO45-Pad26)")
+	(net 61 "unconnected-(U1-IO39-Pad32)")
+	(net 62 "unconnected-(J4-DAT1-Pad8)")
+	(net 63 "unconnected-(J4-SHIELD-Pad11)")
+	(net 64 "unconnected-(J4-DAT3{slash}CD-Pad2)")
+	(net 65 "unconnected-(J4-CMD-Pad3)")
+	(net 66 "unconnected-(J4-DAT0-Pad7)")
+	(net 67 "unconnected-(J4-DAT2-Pad1)")
+	(net 68 "unconnected-(J4-DET_A-Pad10)")
+	(net 69 "unconnected-(J4-CLK-Pad5)")
+	(net 70 "unconnected-(J4-VDD-Pad4)")
+	(net 71 "unconnected-(J4-DET_B-Pad9)")
+	(net 72 "unconnected-(J4-VSS-Pad6)")
+	(net 73 "unconnected-(BZ1-+-Pad1)")
+	(net 74 "unconnected-(BZ1---Pad2)")
+	(net 75 "Net-(P1-VBUS-PadA4)")
+	(net 76 "Net-(P1-GND-PadA1)")
+	(net 77 "unconnected-(P1-CC-PadA5)")
+	(net 78 "unconnected-(P1-SHIELD-PadS1)")
+	(net 79 "unconnected-(P1-VCONN-PadB5)")
+	(net 80 "USB+")
+	(net 81 "USB-")
 	(footprint "Connector_Card:microSD_HC_Hirose_DM3AT-SF-PEJM5"
 		(layer "F.Cu")
@@
 			(size 0.7 1.2)
 			(layers "F.Cu" "F.Mask" "F.Paste")
-			(net 69 "unconnected-(J4-DAT2-Pad1)")
+			(net 67 "unconnected-(J4-DAT2-Pad1)")
 			(pinfunction "DAT2")
 			(pintype "bidirectional")
@@
 			(size 0.7 1.2)
 			(layers "F.Cu" "F.Mask" "F.Paste")
-			(net 66 "unconnected-(J4-DAT3{slash}CD-Pad2)")
+			(net 64 "unconnected-(J4-DAT3{slash}CD-Pad2)")
 			(pinfunction "DAT3/CD")
 			(pintype "bidirectional")
@@
 			(size 0.7 1.2)
 			(layers "F.Cu" "F.Mask" "F.Paste")
-			(net 67 "unconnected-(J4-CMD-Pad3)")
+			(net 65 "unconnected-(J4-CMD-Pad3)")
 			(pinfunction "CMD")
 			(pintype "input")
@@
 			(size 0.7 1.2)
 			(layers "F.Cu" "F.Mask" "F.Paste")
-			(net 72 "unconnected-(J4-VDD-Pad4)")
+			(net 70 "unconnected-(J4-VDD-Pad4)")
 			(pinfunction "VDD")
 			(pintype "power_in")
@@
 			(size 0.7 1.2)
 			(layers "F.Cu" "F.Mask" "F.Paste")
-			(net 71 "unconnected-(J4-CLK-Pad5)")
+			(net 69 "unconnected-(J4-CLK-Pad5)")
 			(pinfunction "CLK")
 			(pintype "input")
@@
 			(size 0.7 1.2)
 			(layers "F.Cu" "F.Mask" "F.Paste")
-			(net 74 "unconnected-(J4-VSS-Pad6)")
+			(net 72 "unconnected-(J4-VSS-Pad6)")
 			(pinfunction "VSS")
 			(pintype "power_in")
@@
 			(size 0.7 1.2)
 			(layers "F.Cu" "F.Mask" "F.Paste")
-			(net 68 "unconnected-(J4-DAT0-Pad7)")
+			(net 66 "unconnected-(J4-DAT0-Pad7)")
 			(pinfunction "DAT0")
 			(pintype "bidirectional")
@@
 			(size 0.7 1.2)
 			(layers "F.Cu" "F.Mask" "F.Paste")
-			(net 64 "unconnected-(J4-DAT1-Pad8)")
+			(net 62 "unconnected-(J4-DAT1-Pad8)")
 			(pinfunction "DAT1")
 			(pintype "bidirectional")
@@
 			(size 0.7 1.2)
 			(layers "F.Cu" "F.Mask" "F.Paste")
-			(net 73 "unconnected-(J4-DET_B-Pad9)")
+			(net 71 "unconnected-(J4-DET_B-Pad9)")
 			(pinfunction "DET_B")
 			(pintype "passive")
@@
 			(size 1 0.8)
 			(layers "F.Cu" "F.Mask" "F.Paste")
-			(net 70 "unconnected-(J4-DET_A-Pad10)")
+			(net 68 "unconnected-(J4-DET_A-Pad10)")
 			(pinfunction "DET_A")
 			(pintype "passive")
@@
 			(size 1 1.2)
 			(layers "F.Cu" "F.Mask" "F.Paste")
-			(net 65 "unconnected-(J4-SHIELD-Pad11)")
+			(net 63 "unconnected-(J4-SHIELD-Pad11)")
 			(pinfunction "SHIELD")
 			(pintype "passive")
@@
 			(size 1 2.8)
 			(layers "F.Cu" "F.Mask" "F.Paste")
-			(net 65 "unconnected-(J4-SHIELD-Pad11)")
+			(net 63 "unconnected-(J4-SHIELD-Pad11)")
 			(pinfunction "SHIELD")
 			(pintype "passive")
@@
 			(size 1 1.2)
 			(layers "F.Cu" "F.Mask" "F.Paste")
-			(net 65 "unconnected-(J4-SHIELD-Pad11)")
+			(net 63 "unconnected-(J4-SHIELD-Pad11)")
 			(pinfunction "SHIELD")
 			(pintype "passive")
@@
 			(size 1.3 1.9)
 			(layers "F.Cu" "F.Mask" "F.Paste")
-			(net 65 "unconnected-(J4-SHIELD-Pad11)")
+			(net 63 "unconnected-(J4-SHIELD-Pad11)")
 			(pinfunction "SHIELD")
 			(pintype "passive")
@@
 			(size 0.3 0.7)
 			(layers "F.Cu" "F.Mask" "F.Paste")
-			(net 78 "Net-(P1-GND-PadA1)")
+			(net 76 "Net-(P1-GND-PadA1)")
 			(pinfunction "GND")
 			(pintype "passive")
@@
 			(size 0.3 0.7)
 			(layers "F.Cu" "F.Mask" "F.Paste")
-			(net 77 "Net-(P1-VBUS-PadA4)")
+			(net 75 "Net-(P1-VBUS-PadA4)")
 			(pinfunction "VBUS")
 			(pintype "passive")
@@
 			(size 0.3 0.7)
 			(layers "F.Cu" "F.Mask" "F.Paste")
-			(net 79 "unconnected-(P1-CC-PadA5)")
+			(net 77 "unconnected-(P1-CC-PadA5)")
 			(pinfunction "CC")
 			(pintype "bidirectional")
@@
 			(size 0.3 0.7)
 			(layers "F.Cu" "F.Mask" "F.Paste")
-			(net 81 "unconnected-(P1-D+-PadA6)")
+			(net 80 "USB+")
 			(pinfunction "D+")
 			(pintype "bidirectional")
@@
 			(size 0.3 0.7)
 			(layers "F.Cu" "F.Mask" "F.Paste")
-			(net 83 "unconnected-(P1-D--PadA7)")
+			(net 81 "USB-")
 			(pinfunction "D-")
 			(pintype "bidirectional")
@@
 			(size 0.3 0.7)
 			(layers "F.Cu" "F.Mask" "F.Paste")
-			(net 77 "Net-(P1-VBUS-PadA4)")
+			(net 75 "Net-(P1-VBUS-PadA4)")
 			(pinfunction "VBUS")
 			(pintype "passive")
@@
 			(size 0.3 0.7)
 			(layers "F.Cu" "F.Mask" "F.Paste")
-			(net 78 "Net-(P1-GND-PadA1)")
+			(net 76 "Net-(P1-GND-PadA1)")
 			(pinfunction "GND")
 			(pintype "passive")
@@
 			(size 0.3 0.7)
 			(layers "F.Cu" "F.Mask" "F.Paste")
-			(net 78 "Net-(P1-GND-PadA1)")
+			(net 76 "Net-(P1-GND-PadA1)")
 			(pinfunction "GND")
 			(pintype "passive")
@@
 			(size 0.3 0.7)
 			(layers "F.Cu" "F.Mask" "F.Paste")
-			(net 77 "Net-(P1-VBUS-PadA4)")
+			(net 75 "Net-(P1-VBUS-PadA4)")
 			(pinfunction "VBUS")
 			(pintype "passive")
@@
 			(size 0.3 0.7)
 			(layers "F.Cu" "F.Mask" "F.Paste")
-			(net 82 "unconnected-(P1-VCONN-PadB5)")
+			(net 79 "unconnected-(P1-VCONN-PadB5)")
 			(pinfunction "VCONN")
 			(pintype "bidirectional")
@@
 			(size 0.3 0.7)
 			(layers "F.Cu" "F.Mask" "F.Paste")
-			(net 77 "Net-(P1-VBUS-PadA4)")
+			(net 75 "Net-(P1-VBUS-PadA4)")
 			(pinfunction "VBUS")
 			(pintype "passive")
@@
 			(size 0.3 0.7)
 			(layers "F.Cu" "F.Mask" "F.Paste")
-			(net 78 "Net-(P1-GND-PadA1)")
+			(net 76 "Net-(P1-GND-PadA1)")
 			(pinfunction "GND")
 			(pintype "passive")
@@
 			(layers "*.Cu" "*.Mask")
 			(remove_unused_layers no)
-			(net 80 "unconnected-(P1-SHIELD-PadS1)")
+			(net 78 "unconnected-(P1-SHIELD-PadS1)")
 			(pinfunction "SHIELD")
 			(pintype "passive")
@@
 			(layers "*.Cu" "*.Mask")
 			(remove_unused_layers no)
-			(net 80 "unconnected-(P1-SHIELD-PadS1)")
+			(net 78 "unconnected-(P1-SHIELD-PadS1)")
 			(pinfunction "SHIELD")
 			(pintype "passive")
@@
 			(layers "*.Cu" "*.Mask")
 			(remove_unused_layers no)
-			(net 80 "unconnected-(P1-SHIELD-PadS1)")
+			(net 78 "unconnected-(P1-SHIELD-PadS1)")
 			(pinfunction "SHIELD")
 			(pintype "passive")
@@
 			(layers "*.Cu" "*.Mask")
 			(remove_unused_layers no)
-			(net 80 "unconnected-(P1-SHIELD-PadS1)")
+			(net 78 "unconnected-(P1-SHIELD-PadS1)")
 			(pinfunction "SHIELD")
 			(pintype "passive")
@@
 			(size 2.2 2.2)
 			(layers "F.Cu" "F.Mask" "F.Paste")
-			(net 75 "unconnected-(BZ1-+-Pad1)")
+			(net 73 "unconnected-(BZ1-+-Pad1)")
 			(pinfunction "+")
 			(pintype "passive")
@@
 			(size 2.2 2.2)
 			(layers "F.Cu" "F.Mask" "F.Paste")
-			(net 76 "unconnected-(BZ1---Pad2)")
+			(net 74 "unconnected-(BZ1---Pad2)")
 			(pinfunction "-")
 			(pintype "passive")
@@
 			(size 1.5 0.9)
 			(layers "F.Cu" "F.Mask" "F.Paste")
-			(net 61 "unconnected-(U1-USB_D--Pad13)")
+			(net 81 "USB-")
 			(pinfunction "USB_D-")
 			(pintype "bidirectional")
@@
 			(size 1.5 0.9)
 			(layers "F.Cu" "F.Mask" "F.Paste")
-			(net 57 "unconnected-(U1-USB_D+-Pad14)")
+			(net 80 "USB+")
 			(pinfunction "USB_D+")
 			(pintype "bidirectional")
@@
 			(size 1.5 0.9)
 			(layers "F.Cu" "F.Mask" "F.Paste")
-			(net 60 "unconnected-(U1-IO10-Pad18)")
+			(net 59 "unconnected-(U1-IO10-Pad18)")
 			(pinfunction "IO10")
 			(pintype "bidirectional")
@@
 			(size 1.5 0.9)
 			(layers "F.Cu" "F.Mask" "F.Paste")
-			(net 58 "unconnected-(U1-IO11-Pad19)")
+			(net 57 "unconnected-(U1-IO11-Pad19)")
 			(pinfunction "IO11")
 			(pintype "bidirectional")
@@
 			(size 1.5 0.9)
 			(layers "F.Cu" "F.Mask" "F.Paste")
-			(net 59 "unconnected-(U1-IO21-Pad23)")
+			(net 58 "unconnected-(U1-IO21-Pad23)")
 			(pinfunction "IO21")
 			(pintype "bidirectional")
@@
 			(size 1.5 0.9)
 			(layers "F.Cu" "F.Mask" "F.Paste")
-			(net 62 "unconnected-(U1-IO45-Pad26)")
+			(net 60 "unconnected-(U1-IO45-Pad26)")
 			(pinfunction "IO45")
 			(pintype "bidirectional")
@@
 			(size 1.5 0.9)
 			(layers "F.Cu" "F.Mask" "F.Paste")
-			(net 63 "unconnected-(U1-IO39-Pad32)")
+			(net 61 "unconnected-(U1-IO39-Pad32)")
 			(pinfunction "IO39")
 			(pintype "bidirectional")

Commit message: added lots of things to main board
Parts:
- removed P1: USB_C_Plug_USB2.0, Connector_USB:USB_C_Receptacle_Amphenol_12401610E4-2A
- added BOOT1: RESET, Button_Switch_SMD:SW_Push_1P1T_NO_CK_KMR2, F.Cu at (66.7, 133.8)
- added C1: 10uF, Capacitor_SMD:C_0805_2012Metric, F.Cu at (58.2, 113.0)
- added C10: 10uF, Capacitor_SMD:C_0805_2012Metric, F.Cu at (58.2, 125.0)
- added C11: 0u1F, Capacitor_SMD:C_0402_1005Metric, F.Cu at (71.7, 122.3)
- added C12: 10uF, Capacitor_SMD:C_0805_2012Metric, F.Cu at (58.2, 128.0)
- added C13: 100nF, Capacitor_SMD:C_0402_1005Metric, F.Cu at (71.7, 124.3)
- added C14: 1uF, Capacitor_SMD:C_0603_1608Metric, F.Cu at (75.1, 123.9)
- added C15: 10uF, Capacitor_SMD:C_0805_2012Metric, F.Cu at (58.2, 131.0)
- added C16: 0u1F, Capacitor_SMD:C_0402_1005Metric, F.Cu at (71.7, 126.2)
- added C2: 10uF, Capacitor_SMD:C_0805_2012Metric, F.Cu at (58.2, 116.0)
- added C3: 0u1F, Capacitor_SMD:C_0402_1005Metric, F.Cu at (71.7, 112.4)
- added C4: 10uF, Capacitor_SMD:C_0805_2012Metric, F.Cu at (58.2, 119.0)
- added C5: 0u1F, Capacitor_SMD:C_0402_1005Metric, F.Cu at (71.7, 114.4)
- added C6: 0u1F, Capacitor_SMD:C_0402_1005Metric, F.Cu at (71.7, 116.4)
- added C7: 0u1F, Capacitor_SMD:C_0402_1005Metric, F.Cu at (71.7, 118.4)
- added C8: 10uF, Capacitor_SMD:C_0805_2012Metric, F.Cu at (58.2, 122.0)
- added C9: 0u1F, Capacitor_SMD:C_0402_1005Metric, F.Cu at (71.7, 120.3)
- added D1: 1N5819WS, Diode_SMD:D_SOD-323, F.Cu at (81.4, 138.7)
- added D2: D_TVS_Small_Filled, Diode_SMD:D_0805_2012Metric, F.Cu at (81.5, 129.6)
- added D3: D_TVS_Small_Filled, Diode_SMD:D_0805_2012Metric, F.Cu at (81.5, 132.7)
- added D4: D_TVS_Small_Filled, Diode_SMD:D_0805_2012Metric, F.Cu at (81.5, 135.7)
- added D5: PWRLED, LED_SMD:LED_0603_1608Metric, F.Cu at (81.3, 141.5)
- added J5: USB_C_Receptacle_USB2.0_16P, Connector_USB:USB_C_Receptacle_GCT_USB4085, F.Cu at (60.8, 79.5)
- added J6: LIPO GND, TestPoint:TestPoint_Pad_4.0x4.0mm, F.Cu at (76.2, 131.1)
- added J7: LIPO PWR, TestPoint:TestPoint_Pad_4.0x4.0mm, F.Cu at (76.2, 137.2)
- added R1: 5k1, Resistor_SMD:R_1206_3216Metric, F.Cu at (53.2, 113.1)
- added R2: 5k1, Resistor_SMD:R_1206_3216Metric, F.Cu at (53.2, 116.4)
- added R3: 75, Resistor_SMD:R_1206_3216Metric, F.Cu at (53.2, 119.7)
- added R4: 10k, Resistor_SMD:R_1206_3216Metric, F.Cu at (53.2, 123.0)
- added R5: 10k, Resistor_SMD:R_1206_3216Metric, F.Cu at (53.2, 126.4)
- added R6: 75, Resistor_SMD:R_1206_3216Metric, F.Cu at (53.2, 129.7)
- added R7: 10k, Resistor_SMD:R_1206_3216Metric, F.Cu at (53.2, 133.0)
- added RESET1: BOOT, Button_Switch_SMD:SW_Push_1P1T_NO_CK_KMR2, F.Cu at (66.7, 138.5)
- added U2: AMS1117-3.3, Package_TO_SOT_SMD:SOT-223-3_TabPin2, F.Cu at (65.3, 115.7)
- added U3: AMS1117-3.3, Package_TO_SOT_SMD:SOT-223-3_TabPin2, F.Cu at (65.3, 124.0)
- moved J4 22.1 mm to (79.9, 87.5), turned to 90 degrees
- moved BZ1 20.0 mm to (59.2, 66.4), turned to 90 degrees
- moved U1 3.71 mm to (73.7, 63.7)
Connections:
- BZ1 pad 1: unconnected-(BZ1-+-Pad1) -> BZR
- BZ1 pad 2: unconnected-(BZ1---Pad2) -> GND
- J1 pad 7: I5 -> SELECT RETURN
- J4 pad 1: unconnected-(J4-DAT2-Pad1) -> SD_DAT2
- J4 pad 10: unconnected-(J4-DET_A-Pad10) -> SD_DET
- J4 pad 11: unconnected-(J4-SHIELD-Pad11) -> GND
- J4 pad 2: unconnected-(J4-DAT3/CD-Pad2) -> SD_DAT3
- J4 pad 3: unconnected-(J4-CMD-Pad3) -> SD_CMD
- J4 pad 4: unconnected-(J4-VDD-Pad4) -> ESP_3V3
- J4 pad 5: unconnected-(J4-CLK-Pad5) -> SD_CLK
- J4 pad 6: unconnected-(J4-VSS-Pad6) -> GND
- J4 pad 7: unconnected-(J4-DAT0-Pad7) -> SD_DAT0
- J4 pad 8: unconnected-(J4-DAT1-Pad8) -> SD_DAT1
- J4 pad 9: unconnected-(J4-DET_B-Pad9) -> SD_DET
- U1 pad 1: Net-(U1-GND-Pad1) -> GND
- U1 pad 2: unconnected-(U1-3V3-Pad2) -> ESP_3V3
- U1 pad 21: unconnected-(U1-IO13-Pad21) -> SELECT RETURN
- U1 pad 22: unconnected-(U1-IO14-Pad22) -> I4
- U1 pad 23: unconnected-(U1-IO21-Pad23) -> I2
- U1 pad 24: unconnected-(U1-IO47-Pad24) -> I3
- U1 pad 25: unconnected-(U1-IO48-Pad25) -> I1
- U1 pad 26: unconnected-(U1-IO45-Pad26) -> I0
- U1 pad 27: unconnected-(U1-IO0-Pad27) -> GPIO0
- U1 pad 28: unconnected-(U1-IO35-Pad28) -> SD_DAT1
- U1 pad 29: unconnected-(U1-IO36-Pad29) -> SD_DAT0
- U1 pad 3: unconnected-(U1-EN-Pad3) -> CHIP_PU
- U1 pad 30: unconnected-(U1-IO37-Pad30) -> SD_CLK
- U1 pad 31: unconnected-(U1-IO38-Pad31) -> SD_DET
- U1 pad 32: unconnected-(U1-IO39-Pad32) -> SD_CMD
- U1 pad 33: unconnected-(U1-IO40-Pad33) -> SD_DAT3
- U1 pad 34: unconnected-(U1-IO41-Pad34) -> SD_DAT2
- U1 pad 40: Net-(U1-GND-Pad1) -> GND
- U1 pad 41: Net-(U1-GND-Pad1) -> GND

Commit message: more main board stuff
Parts:
- added R10: 10k, Resistor_SMD:R_1206_3216Metric, F.Cu at (82.4, 108.8)
- added R12: 10k, Resistor_SMD:R_1206_3216Metric, F.Cu at (82.4, 112.1)
- added R13: 10k, Resistor_SMD:R_1206_3216Metric, F.Cu at (82.4, 115.4)
- added R8: 10k, Resistor_SMD:R_1206_3216Metric, F.Cu at (82.4, 102.2)
- added R9: 10k, Resistor_SMD:R_1206_3216Metric, F.Cu at (82.4, 105.5)
- BZ1: footprint Buzzer_Beeper:Buzzer_Mallory_AST1109MLTRQ -> Buzzer_Beeper:MagneticBuzzer_Kingstate_KCG0601
- moved BZ1 38.2 mm to (58.3, 104.6), turned to 0 degrees
- moved U1 3.76 mm to (70.0, 63.7)
- moved J5 0.84 mm to (60.0, 79.4)
Connections:
- J2 pad 1: unconnected-(J2-Pin_1-Pad1) -> DATA8
- J2 pad 2: unconnected-(J2-Pin_2-Pad2) -> DATA9
- J2 pad 3: unconnected-(J2-Pin_3-Pad3) -> DATA10
- J2 pad 4: unconnected-(J2-Pin_4-Pad4) -> DATA11
- J2 pad 5: unconnected-(J2-Pin_5-Pad5) -> DATA12
- J2 pad 6: unconnected-(J2-Pin_6-Pad6) -> DATA13
- J2 pad 7: unconnected-(J2-Pin_7-Pad7) -> DATA14
- J2 pad 8: unconnected-(J2-Pin_8-Pad8) -> DATA15
- J3 pad 1: unconnected-(J3-Pin_1-Pad1) -> DATA7
- J3 pad 2: unconnected-(J3-Pin_2-Pad2) -> DATA6
- J3 pad 3: unconnected-(J3-Pin_3-Pad3) -> DATA5
- J3 pad 4: unconnected-(J3-Pin_4-Pad4) -> DATA4
- J3 pad 5: unconnected-(J3-Pin_5-Pad5) -> DATA3
- J3 pad 6: unconnected-(J3-Pin_6-Pad6) -> DATA2
- J3 pad 7: unconnected-(J3-Pin_7-Pad7) -> DATA1
- J3 pad 8: unconnected-(J3-Pin_8-Pad8) -> DATA0
- U1 pad 10: unconnected-(U1-IO17-Pad10) -> DATA11
- U1 pad 11: unconnected-(U1-IO18-Pad11) -> DATA12
- U1 pad 12: unconnected-(U1-IO8-Pad12) -> DATA13
- U1 pad 15: unconnected-(U1-IO3-Pad15) -> DATA14
- U1 pad 16: unconnected-(U1-IO46-Pad16) -> DATA15
- U1 pad 35: unconnected-(U1-IO42-Pad35) -> DATA7
- U1 pad 36: unconnected-(U1-RXD0-Pad36) -> DATA6
- U1 pad 37: unconnected-(U1-TXD0-Pad37) -> DATA5
- U1 pad 38: unconnected-(U1-IO2-Pad38) -> DATA4
- U1 pad 39: unconnected-(U1-IO1-Pad39) -> DATA3
- U1 pad 4: unconnected-(U1-IO4-Pad4) -> DATA0
- U1 pad 5: unconnected-(U1-IO5-Pad5) -> DATA1
- U1 pad 6: unconnected-(U1-IO6-Pad6) -> DATA2
- U1 pad 7: unconnected-(U1-IO7-Pad7) -> DATA8
- U1 pad 8: unconnected-(U1-IO15-Pad8) -> DATA9
- U1 pad 9: unconnected-(U1-IO16-Pad9) -> DATA10

Commit message: finished main board
Parts:
- removed RESET1: BOOT, Button_Switch_SMD:SW_Push_1P1T_NO_CK_KMR2
- added D6: PWRLED, LED_SMD:LED_0603_1608Metric, F.Cu at (87.9, 108.9)
- added Enable: En_B, TestPoint:TestPoint_Pad_1.5x1.5mm, F.Cu at (87.1, 114.1)
- added J8: En_A, TestPoint:TestPoint_Pad_1.5x1.5mm, F.Cu at (87.1, 118.5)
- added Q1: MMBT2222A, Package_TO_SOT_SMD:SOT-23W_Handsoldering, F.Cu at (55.4, 117.2)
- U3: value AMS1117-3.3 -> AMS1117-5.0
- moved C15 72.3 mm to (59.0, 58.8), turned to 90 degrees
- moved R7 71.8 mm to (56.7, 61.3), turned to -90 degrees
- moved C16 69.7 mm to (57.4, 58.0), turned to 90 degrees
- moved D4 65.6 mm to (56.6, 75.0), turned to 180 degrees
- moved D3 64.7 mm to (56.6, 72.9), turned to 180 degrees
- moved C14 64.0 mm to (58.7, 62.1), turned to 90 degrees
- moved D1 52.8 mm to (59.3, 90.8), turned to 180 degrees
- moved D2 46.5 mm to (59.4, 88.8)
- moved D5 40.6 mm to (88.0, 101.4), turned to -90 degrees
- moved - 40.0 mm to (54.8, 103.4), turned to 90 degrees
- moved R6 38.9 mm to (86.0, 108.8), turned to -90 degrees
- moved R3 37.7 mm to (86.0, 101.3), turned to -90 degrees
- moved R2 36.5 mm to (63.4, 81.4)
- moved C12 32.0 mm to (70.9, 98.7), turned to 180 degrees
- moved J1 31.9 mm to (78.7, 118.7)
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- renumbered J6 to +, J7 to -, BOOT1 to BOOT, BZ1 to BZ, U1 to ESP32-S3-WROOM-1
Connections:
- BOOT pad 1: GND -> LIPO GND
- BZ pad 2: GND -> LIPO GND
- C1 pad 2: GND -> LIPO GND
- C10 pad 2: GND -> LIPO GND
- C11 pad 2: GND -> LIPO GND
- C12 pad 2: GND -> LIPO GND
- C13 pad 2: GND -> LIPO GND
- C14 pad 2: GND -> LIPO GND
- C15 pad 2: GND -> LIPO GND
- C16 pad 2: GND -> LIPO GND
- C2 pad 2: GND -> LIPO GND
- C3 pad 2: GND -> LIPO GND
- C4 pad 2: GND -> LIPO GND
- C5 pad 2: GND -> LIPO GND
- C6 pad 2: GND -> LIPO GND
- C7 pad 2: GND -> LIPO GND
- C8 pad 2: GND -> LIPO GND
- C9 pad 2: GND -> LIPO GND
- D2 pad 2: GND -> LIPO GND
- D3 pad 2: GND -> LIPO GND
- D4 pad 2: GND -> LIPO GND
- D5 pad 1: GND -> LIPO GND
- ESP32-S3-WROOM-1 pad 1: GND -> LIPO GND
- ESP32-S3-WROOM-1 pad 18: unconnected-(U1-IO10-Pad18) -> BZR
- ESP32-S3-WROOM-1 pad 20: unconnected-(U1-IO12-Pad20) -> HATS_ENABLE
- ESP32-S3-WROOM-1 pad 23: I2 -> I3
- ESP32-S3-WROOM-1 pad 24: I3 -> I2
- ESP32-S3-WROOM-1 pad 28: SD_DAT1 -> SD_DAT2
- ESP32-S3-WROOM-1 pad 29: SD_DAT0 -> SD_DAT3
- ESP32-S3-WROOM-1 pad 30: SD_CLK -> SD_CMD
- ESP32-S3-WROOM-1 pad 32: SD_CMD -> SD_CLK
- ESP32-S3-WROOM-1 pad 33: SD_DAT3 -> SD_DAT0
- ESP32-S3-WROOM-1 pad 34: SD_DAT2 -> SD_DAT1
- ESP32-S3-WROOM-1 pad 40: GND -> LIPO GND
- ESP32-S3-WROOM-1 pad 41: GND -> LIPO GND
- J1 pad 1: GND -> LIPO GND
- J1 pad 8: +5V -> Net-(J1-Pin_8)
- J4 pad 11: GND -> LIPO GND
- J4 pad 6: GND -> LIPO GND
- J5 pad A1: GND -> LIPO GND
- J5 pad A12: GND -> LIPO GND
- J5 pad B1: GND -> LIPO GND
- J5 pad B12: GND -> LIPO GND
- J5 pad S1: GND -> LIPO GND
- R1 pad 2: GND -> LIPO GND
- R2 pad 2: GND -> LIPO GND
- R5 pad 2: CHIP_PU -> Net-(J8-Pin_1)
- R6 pad 2: GND -> Net-(D6-A)
- U2 pad 1: GND -> LIPO GND
- U3 pad 1: GND -> LIPO GND
Routing:
- net ESP_3V3: track 0.00 -> 176.0 mm, vias 0 -> 4
- net LIPO GND: track 0.00 -> 93.7 mm, vias 0 -> 36
- net CHIP_PU: track 0.00 -> 87.1 mm, vias 0 -> 2
- net VCC_5V: track 0.00 -> 65.8 mm
- net HATS_ENABLE: track 0.00 -> 52.0 mm, vias 0 -> 2
- net I0: track 0.00 -> 51.7 mm, vias 0 -> 1
- net LIPO PWR: track 0.00 -> 50.6 mm
- net I1: track 0.00 -> 50.3 mm, vias 0 -> 1
- net I2: track 0.00 -> 49.0 mm, vias 0 -> 1
- net GPIO0: track 0.00 -> 48.6 mm
- net I3: track 0.00 -> 47.8 mm, vias 0 -> 1
- net I4: track 0.00 -> 46.3 mm, vias 0 -> 1
- net SELECT RETURN: track 0.00 -> 46.0 mm, vias 0 -> 1
- net SD_DET: track 0.00 -> 40.6 mm, vias 0 -> 2
- net SD_DAT1: track 0.00 -> 37.8 mm
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- added copper zone on B.Cu, net LIPO GND
- added copper zone on F.Cu, net LIPO GND
Other:
- board size 38.1 x 101.6 mm -> 38.1 x 73.8 mm
- board text added: "3V3 PWR"
- board text added: "5V PWR"
- board text added: "Power In"
