File: hardware/MainBoard/MainBoard.kicad_sch (KiCad schematic)
At the start: 27 parts, among them J1 Conn_02x16_Top_Bottom, J2 Conn_02x16_Top_Bottom, J7 Conn_02x16_Top_Bottom, Q1 MMBT2222A, U1 ESP32-S3-WROOM-1, U2 AMS1117-3.3, U3 AMS1117-5.0

Commit message: finished 1x1 main board
Parts:
- +1: value LIPO GND -> LIPO PWR
- -1: value LIPO PWR -> LIPO GND
Connections:
- net CONN_17 is gone; now on net BZR: J1.18 (Pin_18), J2.3 (Pin_3)
- net SD_DET is gone; now on net CONN_11: U1.31 (IO38)
- net VCC_5V is gone; now on net CONN_VCC: C10.1, C11.1, Q1.3 (C), R3.1, U3.2 (VO)
- net CONN_0: now also U1.14 (USB_D+)
- net CONN_10: now also U1.30 (IO37)
- net CONN_14: now also U1.32 (IO39); no longer I2C_DAT1.1 (Pin_1), U1.19 (IO11)
- net CONN_16: now also I2C_DAT1.1 (Pin_1), U1.19 (IO11)
- net CONN_2: now also U1.13 (USB_D-)
- net CONN_22: no longer U1.13 (USB_D-)
- net CONN_23: no longer U1.14 (USB_D+)
- net CONN_24: no longer U1.28 (IO35)
- net CONN_25: no longer U1.29 (IO36)
- net CONN_26: no longer U1.30 (IO37)
- net CONN_27: no longer U1.32 (IO39)
- net CONN_6: now also U1.28 (IO35)
- net CONN_7: now also U1.29 (IO36)
- net DATA0: now also J7.15 (Pin_15); no longer J7.1 (Pin_1)
- net DATA1: now also J7.14 (Pin_14); no longer J7.2 (Pin_2)
- net DATA10: now also J7.2 (Pin_2); no longer J7.11 (Pin_11)
- net DATA11: now also J7.3 (Pin_3); no longer J7.12 (Pin_12)
- net DATA12: now also J7.4 (Pin_4); no longer J7.13 (Pin_13)
- net DATA13: now also J7.5 (Pin_5); no longer J7.14 (Pin_14)
- net DATA14: now also J7.16 (Pin_16); no longer J7.15 (Pin_15)
- net DATA15: now also J7.17 (Pin_17); no longer J7.16 (Pin_16)
- net DATA2: now also J7.13 (Pin_13); no longer J7.3 (Pin_3)
- net DATA3: now also J7.12 (Pin_12); no longer J7.4 (Pin_4)
- net DATA4: now also J7.11 (Pin_11); no longer J7.5 (Pin_5)
- net DATA5: now also J7.10 (Pin_10); no longer J7.6 (Pin_6)
- net DATA6: now also J7.9 (Pin_9); no longer J7.7 (Pin_7)
- net DATA8: now also J7.7 (Pin_7); no longer J7.9 (Pin_9)
- net DATA9: now also J7.1 (Pin_1); no longer J7.10 (Pin_10)
- net INDEX0: now also J7.26 (Pin_26); no longer J7.30 (Pin_30)
- net INDEX1: now also J7.27 (Pin_27); no longer J7.29 (Pin_29)
- net INDEX3: now also J7.29 (Pin_29); no longer J7.27 (Pin_27)
- net INDEX4: now also J7.30 (Pin_30); no longer J7.26 (Pin_26)
- net CONN_3V renamed LIPO PWR
