File: hardware/MainBoard/peripherals.kicad_sch (KiCad schematic)
At the start: 24 parts, among them J1 USB_C_Receptacle_USB2.0_16P, J2 En_A, J3 En_B, J4 Micro_SD_Card_Det2

Commit message: started wiring main boards
Parts:
- renumbered C4 to C12, C7 to C14, C14 to C15, C10 to C16, D1 to D3, D2 to D4, D3 to D5, D4 to D6, J1 to J3, J2 to J4, J3 to J5, J4 to J6, R4 to R10, R5 to R12, R2 to R4, R3 to R5, R7 to R6, R8 to R7, R9 to R8, R10 to R9
Changed lines of the file:
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@@
 		(dnp no)
 		(fields_autoplaced yes)
-		(property "Reference" "R3"
+		(property "Reference" "R5"
 			(at 57.15 30.4799 0)
 			(effects
@@
 			(project "MainBoard"
 				(path "/988df97c-fca1-40e2-af98-331e3f3f354f/0083cdc5-b2ac-4b53-bbf9-3ad68cb40dda"
-					(reference "R3")
+					(reference "R5")
 					(unit 1)
 				)
@@
 		(dnp no)
 		(fields_autoplaced yes)
-		(property "Reference" "J1"
+		(property "Reference" "J3"
 			(at 35.56 29.21 0)
 			(effects
@@
 			(project "MainBoard"
 				(path "/988df97c-fca1-40e2-af98-331e3f3f354f/0083cdc5-b2ac-4b53-bbf9-3ad68cb40dda"
-					(reference "J1")
+					(reference "J3")
 					(unit 1)
 				)
@@
 		(dnp no)
 		(fields_autoplaced yes)
-		(property "Reference" "J4"
+		(property "Reference" "J6"
 			(at 155.575 68.58 0)
 			(effects
@@
 			(project "MainBoard"
 				(path "/988df97c-fca1-40e2-af98-331e3f3f354f/0083cdc5-b2ac-4b53-bbf9-3ad68cb40dda"
-					(reference "J4")
+					(reference "J6")
 					(unit 1)
 				)
@@
 		(dnp no)
 		(fields_autoplaced yes)
-		(property "Reference" "R5"
+		(property "Reference" "R12"
 			(at 140.97 30.4799 0)
 			(effects
@@
 			(project "MainBoard"
 				(path "/988df97c-fca1-40e2-af98-331e3f3f354f/0083cdc5-b2ac-4b53-bbf9-3ad68cb40dda"
-					(reference "R5")
+					(reference "R12")
 					(unit 1)
 				)
@@
 		(on_board yes)
 		(dnp no)
-		(property "Reference" "R9"
+		(property "Reference" "R8"
 			(at 115.57 76.1999 0)
 			(effects
@@
 			(project "MainBoard"
 				(path "/988df97c-fca1-40e2-af98-331e3f3f354f/0083cdc5-b2ac-4b53-bbf9-3ad68cb40dda"
-					(reference "R9")
+					(reference "R8")
 					(unit 1)
 				)
@@
 		(dnp no)
 		(fields_autoplaced yes)
-		(property "Reference" "C4"
+		(property "Reference" "C12"
 			(at 82.55 62.2299 0)
 			(effects
@@
 			(project "MainBoard"
 				(path "/988df97c-fca1-40e2-af98-331e3f3f354f/0083cdc5-b2ac-4b53-bbf9-3ad68cb40dda"
-					(reference "C4")
+					(reference "C12")
 					(unit 1)
 				)
@@
 		(on_board yes)
 		(dnp no)
-		(property "Reference" "J3"
+		(property "Reference" "J5"
 			(at 145.542 44.196 0)
 			(effects
@@
 			(project "MainBoard"
 				(path "/988df97c-fca1-40e2-af98-331e3f3f354f/0083cdc5-b2ac-4b53-bbf9-3ad68cb40dda"
-					(reference "J3")
+					(reference "J5")
 					(unit 1)
 				)
@@
 		(on_board yes)
 		(dnp no)
-		(property "Reference" "D3"
+		(property "Reference" "D5"
 			(at 62.738 61.214 90)
 			(effects
@@
 			(project "MainBoard"
 				(path "/988df97c-fca1-40e2-af98-331e3f3f354f/0083cdc5-b2ac-4b53-bbf9-3ad68cb40dda"
-					(reference "D3")
+					(reference "D5")
 					(unit 1)
 				)
@@
 		(dnp no)
 		(fields_autoplaced yes)
-		(property "Reference" "R2"
+		(property "Reference" "R4"
 			(at 55.88 71.1199 0)
 			(effects
@@
 			(project "MainBoard"
 				(path "/988df97c-fca1-40e2-af98-331e3f3f354f/0083cdc5-b2ac-4b53-bbf9-3ad68cb40dda"
-					(reference "R2")
+					(reference "R4")
 					(unit 1)
 				)
@@
 		(dnp no)
 		(fields_autoplaced yes)
-		(property "Reference" "#PWR015"
+		(property "Reference" "#PWR016"
 			(at 116.84 128.27 0)
 			(effects
@@
 			(project "MainBoard"
 				(path "/988df97c-fca1-40e2-af98-331e3f3f354f/0083cdc5-b2ac-4b53-bbf9-3ad68cb40dda"
-					(reference "#PWR015")
+					(reference "#PWR016")
 					(unit 1)
 				)
@@
 		(dnp no)
 		(fields_autoplaced yes)
-		(property "Reference" "C10"
+		(property "Reference" "C16"
 			(at 162.56 48.2599 0)
 			(effects
@@
 			(project "MainBoard"
 				(path "/988df97c-fca1-40e2-af98-331e3f3f354f/0083cdc5-b2ac-4b53-bbf9-3ad68cb40dda"
-					(reference "C10")
+					(reference "C16")
 					(unit 1)
 				)
@@
 		(dnp no)
 		(fields_autoplaced yes)
-		(property "Reference" "#PWR02"
+		(property "Reference" "#PWR011"
 			(at 40.64 85.09 0)
 			(effects
@@
 			(project "MainBoard"
 				(path "/988df97c-fca1-40e2-af98-331e3f3f354f/0083cdc5-b2ac-4b53-bbf9-3ad68cb40dda"
-					(reference "#PWR02")
+					(reference "#PWR011")
 					(unit 1)
 				)
@@
 		(dnp no)
 		(fields_autoplaced yes)
-		(property "Reference" "R4"
+		(property "Reference" "R10"
 			(at 123.19 30.4799 0)
 			(effects
@@
 			(project "MainBoard"
 				(path "/988df97c-fca1-40e2-af98-331e3f3f354f/0083cdc5-b2ac-4b53-bbf9-3ad68cb40dda"
-					(reference "R4")
+					(reference "R10")
 					(unit 1)
 				)
@@
 		(dnp no)
 		(fields_autoplaced yes)
-		(property "Reference" "#PWR016"
+		(property "Reference" "#PWR017"
 			(at 130.81 123.19 0)
 			(effects
@@
 			(project "MainBoard"
 				(path "/988df97c-fca1-40e2-af98-331e3f3f354f/0083cdc5-b2ac-4b53-bbf9-3ad68cb40dda"
-					(reference "#PWR016")
+					(reference "#PWR017")
 					(unit 1)
 				)
@@
 		(on_board yes)
 		(dnp no)
-		(property "Reference" "D1"
+		(property "Reference" "D3"
 			(at 55.88 60.96 90)
 			(effects
@@
 			(project "MainBoard"
 				(path "/988df97c-fca1-40e2-af98-331e3f3f354f/0083cdc5-b2ac-4b53-bbf9-3ad68cb40dda"
-					(reference "D1")
+					(reference "D3")
 					(unit 1)
 				)
@@
 		(dnp no)
 		(fields_autoplaced yes)
-		(property "Reference" "#PWR011"
+		(property "Reference" "#PWR018"
 			(at 158.75 60.96 0)
 			(effects
@@
 			(project "MainBoard"
 				(path "/988df97c-fca1-40e2-af98-331e3f3f354f/0083cdc5-b2ac-4b53-bbf9-3ad68cb40dda"
-					(reference "#PWR011")
+					(reference "#PWR018")
 					(unit 1)
 				)
@@
 		(on_board yes)
 		(dnp no)
-		(property "Reference" "R7"
+		(property "Reference" "R6"
 			(at 102.87 78.7399 0)
 			(effects
@@
 			(project "MainBoard"
 				(path "/988df97c-fca1-40e2-af98-331e3f3f354f/0083cdc5-b2ac-4b53-bbf9-3ad68cb40dda"
-					(reference "R7")
+					(reference "R6")
 					(unit 1)
 				)
@@
 		(dnp no)
 		(fields_autoplaced yes)
-		(property "Reference" "D2"
+		(property "Reference" "D4"
 			(at 66.3575 30.48 0)
 			(effects
@@
 			(project "MainBoard"
 				(path "/988df97c-fca1-40e2-af98-331e3f3f354f/0083cdc5-b2ac-4b53-bbf9-3ad68cb40dda"
-					(reference "D2")
+					(reference "D4")
 					(unit 1)
 				)
@@
 		(on_board yes)
 		(dnp no)
-		(property "Reference" "D4"
+		(property "Reference" "D6"
 			(at 67.564 60.96 90)
 			(effects
@@
 			(project "MainBoard"
 				(path "/988df97c-fca1-40e2-af98-331e3f3f354f/0083cdc5-b2ac-4b53-bbf9-3ad68cb40dda"
-					(reference "D4")
+					(reference "D6")
 					(unit 1)
 				)
@@
 		(dnp no)
 		(fields_autoplaced yes)
-		(property "Reference" "#PWR03"
+		(property "Reference" "#PWR012"
 			(at 54.61 20.32 0)
 			(effects
@@
 			(project "MainBoard"
 				(path "/988df97c-fca1-40e2-af98-331e3f3f354f/0083cdc5-b2ac-4b53-bbf9-3ad68cb40dda"
-					(reference "#PWR03")
+					(reference "#PWR012")
 					(unit 1)
 				)
@@
 		(dnp no)
 		(fields_autoplaced yes)
-		(property "Reference" "C7"
+		(property "Reference" "C14"
 			(at 120.65 44.4499 0)
 			(effects
@@
 			(project "MainBoard"
 				(path "/988df97c-fca1-40e2-af98-331e3f3f354f/0083cdc5-b2ac-4b53-bbf9-3ad68cb40dda"
-					(reference "C7")
+					(reference "C14")
 					(unit 1)
 				)
@@
 		(dnp no)
 		(fields_autoplaced yes)
-		(property "Reference" "#PWR09"
+		(property "Reference" "#PWR013"
 			(at 78.74 109.22 0)
 			(effects
@@
 			(project "MainBoard"
 				(path "/988df97c-fca1-40e2-af98-331e3f3f354f/0083cdc5-b2ac-4b53-bbf9-3ad68cb40dda"
-					(reference "#PWR09")
+					(reference "#PWR013")
 					(unit 1)
 				)
@@
 		(on_board yes)
 		(dnp no)
-		(property "Reference" "J2"
+		(property "Reference" "J4"
 			(at 146.05 34.036 0)
 			(effects
@@
 			(project "MainBoard"
 				(path "/988df97c-fca1-40e2-af98-331e3f3f354f/0083cdc5-b2ac-4b53-bbf9-3ad68cb40dda"
-					(reference "J2")
+					(reference "J4")
 					(unit 1)
 				)
@@
 		(on_board yes)
 		(dnp no)
-		(property "Reference" "R10"
+		(property "Reference" "R9"
 			(at 115.57 104.1401 0)
 			(effects
@@
 			(project "MainBoard"
 				(path "/988df97c-fca1-40e2-af98-331e3f3f354f/0083cdc5-b2ac-4b53-bbf9-3ad68cb40dda"
-					(reference "R10")
+					(reference "R9")
 					(unit 1)
 				)
@@
 		(on_board yes)
 		(dnp no)
-		(property "Reference" "R8"
+		(property "Reference" "R7"
 			(at 102.87 101.6001 0)
 			(effects
@@
 			(project "MainBoard"
 				(path "/988df97c-fca1-40e2-af98-331e3f3f354f/0083cdc5-b2ac-4b53-bbf9-3ad68cb40dda"
-					(reference "R8")
+					(reference "R7")
 					(unit 1)
 				)
@@
 		(on_board yes)
 		(dnp no)
-		(property "Reference" "C14"
+		(property "Reference" "C15"
 			(at 120.65 118.364 0)
 			(effects
@@
 			(project "MainBoard"
 				(path "/988df97c-fca1-40e2-af98-331e3f3f354f/0083cdc5-b2ac-4b53-bbf9-3ad68cb40dda"
-					(reference "C14")
+					(reference "C15")
 					(unit 1)
 				)
@@
 		(dnp no)
 		(fields_autoplaced yes)
-		(property "Reference" "#PWR07"
+		(property "Reference" "#PWR015"
 			(at 116.84 60.96 0)
 			(effects
@@
 			(project "MainBoard"
 				(path "/988df97c-fca1-40e2-af98-331e3f3f354f/0083cdc5-b2ac-4b53-bbf9-3ad68cb40dda"
-					(reference "#PWR07")
-					(unit 1)
-				)
+					(reference "#PWR015")
+					(unit 1)
+				)

Commit message: finished 1x1 main board
Connections:
- net VCC_3V3: no longer C12.1, D4.1 (K)
- new net VCC_5V: C12.1, D4.1 (K)
Changed lines of the file:
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@@
 		)
 	)
-	(global_label "VCC_3V3"
+	(global_label "VCC_5V"
 		(shape input)
 		(at 80.01 26.67 0)
@@
 		)
 		(property "Intersheetrefs" "${INTERSHEET_REFS}"
-			(at 86.6636 26.67 0)
+			(at 85.9379 26.67 0)
 			(effects
 				(font

Commit message: added voltage switcher - still needs to be routed
Connections:
- net VCC_5V renamed VBUS
Changed lines of the file:
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@@
 		)
 	)
-	(global_label "VCC_5V"
+	(global_label "VBUS"
 		(shape input)
 		(at 80.01 26.67 0)
@@
 		)
 		(property "Intersheetrefs" "${INTERSHEET_REFS}"
-			(at 85.9379 26.67 0)
+			(at 84.7405 26.67 0)
 			(effects
 				(font
